File: pcb/FabScan-Shield_v10.sch (EAGLE design)
At the start: 37 parts, among them T1 BC547, T2 IRLML2502, X1 PASSER, X2 PASSER

Commit message: upated schematics
Other:
- note added: "Arduino"
- note added: "Pololu A4988 or StepStick"
- moved on the sheet: D4, D5, LASER-1, LASER-2, LED-1, LED-2, R4, R5, R6, T1, T2, VMOT-1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

Commit message: updated schematic and layout files
Other:
- note added: "Released under the Creative Commons Attribution Share-Alike License"
- note added: "http://creativecommons.org/licenses/by-sa/4.0/"
- note removed: "Released under the Creative Commons Attribution Share-Alike 3.0 License"
- note removed: "http://creativecommons.org/licenses/by-sa/3.0/"
Changed lines of the file:
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@@
 <?xml version="1.0" encoding="utf-8"?>
 <!DOCTYPE eagle SYSTEM "eagle.dtd">
-<eagle version="6.3">
+<eagle version="6.6.0">
 <drawing>
 <settings>
@@
 <setting verticaltext="up"/>
 </settings>
-<grid distance="0.05" unitdist="inch" unit="inch" style="lines" multiple="1" display="yes" altdistance="0.01" altunitdist="inch" altunit="inch"/>
+<grid distance="0.1" unitdist="inch" unit="inch" style="lines" multiple="1" display="no" altdistance="0.01" altunitdist="inch" altunit="inch"/>
 <layers>
 <layer number="1" name="Top" color="4" fill="1" visible="no" active="no"/>
@@
 <plain>
 <wire x1="33.02" y1="149.86" x2="35.687" y2="149.86" width="0.8128" layer="94"/>
-<text x="161.29" y="34.29" size="1.27" layer="95">Released under the Creative Commons Attribution Share-Alike 3.0 License</text>
-<text x="161.29" y="31.75" size="1.27" layer="95">http://creativecommons.org/licenses/by-sa/3.0/</text>
+<text x="161.29" y="34.29" size="1.27" layer="95">Released under the Creative Commons Attribution Share-Alike License</text>
+<text x="161.29" y="31.75" size="1.27" layer="95">http://creativecommons.org/licenses/by-sa/4.0/</text>
 <text x="161.29" y="27.94" size="1.27" layer="95">Designed by Andreas Watterott (Watterott electronic)</text>
 <text x="161.29" y="41.91" size="2.54" layer="95">Further Infos: http://hci.rwth-aachen.de/fabscan</text>
