File: pcb/FabScan-Shield_v10.sch (EAGLE design)
At the start: 37 parts, among them T1 BC547, T2 IRLML2502, X1 PASSER, X2 PASSER

Commit message: cleaned up schematics and layout
Changed lines of the file:
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@@
 <setting verticaltext="up"/>
 </settings>
-<grid distance="0.1" unitdist="inch" unit="inch" style="lines" multiple="1" display="no" altdistance="0.01" altunitdist="inch" altunit="inch"/>
+<grid distance="0.05" unitdist="inch" unit="inch" style="lines" multiple="1" display="yes" altdistance="0.025" altunitdist="inch" altunit="inch"/>
 <layers>
 <layer number="1" name="Top" color="4" fill="1" visible="no" active="no"/>
@@
 </classes>
 <parts>
-<part name="FRAME1" library="frames" deviceset="A4L-LOC" device=""/>
 <part name="GND4" library="supply1" deviceset="GND" device=""/>
 <part name="X1" library="SMD" deviceset="PASSER" device=""/>
@@
 <part name="GND21" library="supply1" deviceset="GND" device=""/>
 <part name="R6" library="rcl" deviceset="R-EU_" device="R0603" value="47k"/>
+<part name="FRAME1" library="we-symbol" deviceset="FRAME-A4L" device=""/>
 </parts>
 <sheets>
@@
 <plain>
 <wire x1="33.02" y1="149.86" x2="35.687" y2="149.86" width="0.8128" layer="94"/>
-<text x="161.29" y="34.29" size="1.27" layer="95">Released under the Creative Commons Attribution Share-Alike License</text>
-<text x="161.29" y="31.75" size="1.27" layer="95">http://creativecommons.org/licenses/by-sa/4.0/</text>
-<text x="161.29" y="27.94" size="1.27" layer="95">Designed by Andreas Watterott (Watterott electronic)</text>
-<text x="161.29" y="41.91" size="2.54" layer="95">Further Infos: http://hci.rwth-aachen.de/fabscan</text>
-<text x="161.29" y="25.4" size="1.27" layer="95">Based on the work of Francis Engelmann and Sebastian Setz</text>
+<text x="162.56" y="21.59" size="1.27" layer="95">Released under the Creative Commons Attribution Share-Alike License</text>
+<text x="162.56" y="19.05" size="1.27" layer="95">http://creativecommons.org/licenses/by-sa/4.0/</text>
+<text x="162.56" y="15.24" size="1.27" layer="95">Designed by Andreas Watterott (Watterott electronic)</text>
+<text x="162.56" y="25.4" size="2.54" layer="95">Further Infos: http://hci.rwth-aachen.de/fabscan</text>
+<text x="162.56" y="12.7" size="1.27" layer="95">Based on the work of Francis Engelmann and Sebastian Setz</text>
 <text x="209.55" y="158.75" size="2.54" layer="95">Servos</text>
 <text x="189.23" y="158.75" size="2.54" layer="95">Steppers</text>
@@
 </plain>
 <instances>
-<instance part="FRAME1" gate="G$1" x="0" y="0" smashed="yes">
-<attribute name="DRAWING_NAME" x="217.17" y="15.24" size="2.54" layer="94" font="vector"/>
-<attribute name="LAST_DATE_TIME" x="217.17" y="10.16" size="2.286" layer="94" font="vector"/>
-<attribute name="SHEET" x="230.505" y="5.08" size="2.54" layer="94" font="vector"/>
-</instance>
 <instance part="GND4" gate="1" x="106.68" y="149.86" smashed="yes" rot="R90">
 <attribute name="VALUE" x="109.22" y="147.32" size="1.778" layer="96" rot="R90"/>
 </instance>
-<instance part="X1" gate="G$1" x="166.37" y="19.05"/>
-<instance part="X2" gate="G$1" x="173.99" y="19.05"/>
+<instance part="X1" gate="G$1" x="165.1" y="7.62" smashed="yes"/>
+<instance part="X2" gate="G$1" x="170.18" y="7.62" smashed="yes"/>
 <instance part="GND8" gate="1" x="157.48" y="129.54" smashed="yes">
 <attribute name="VALUE" x="154.94" y="127" size="1.778" layer="96"/>
@@
 <attribute name="VALUE" x="31.75" y="146.05" size="1.778" layer="96"/>
 </instance>
-<instance part="LOGO2" gate="G$1" x="201.93" y="19.05"/>
+<instance part="LOGO2" gate="G$1" x="208.28" y="7.62"/>
 <instance part="A1" gate="G$1" x="62.23" y="127"/>
 <instance part="GND14" gate="1" x="34.29" y="132.08" smashed="yes" rot="R270">
@@
 <attribute name="VALUE" x="77.978" y="64.643" size="1.778" layer="96" rot="MR180"/>
 </instance>
+<instance part="FRAME1" gate="G$1" x="0" y="0"/>
 </instances>
 <busses>
