File: pcb/FabScan-Shield_v10.brd (EAGLE design)
At the start: 68.6 x 53.3 mm, 37 parts, among them T1 BC547, T2 IRLML2502, X1 PASSER, X2 PASSER

Commit message: updated layout and schematics
Other:
- board text added: "Silkscreen: 51 tDocu"
